Commit message: copy

File: assembly_gym/shapes/cube06.urdf (robot description, URDF)
Before this commit: robot block_t, 1 links, 0 joints
Links:
- link block_t_base_link: mass 1 -> 0.3; geometry collision box size=0.6 0.6 0.6; visual box size=0.6 0.6 0.6

File: assembly_gym/shapes/cube1.urdf (robot description, URDF)
Before this commit: robot block_t, 1 links, 0 joints
Links:
- link block_t_base_link: mass 1 -> 0.3; geometry collision box size=1.0 1.0 1.0; visual box size=1.0 1.0 1.0

File: assembly_gym/shapes/hexagon.urdf (robot description, URDF)
Before this commit: robot block_t, 1 links, 0 joints
Links:
- link block_t_base_link: geometry collision mesh filename=package://blocks/hexagon.stl; visual mesh filename=package://blocks/hexagon.stl
